File: USB 3.0 to Sata.kicad_sch (KiCad schematic)
At the start: 9 parts, among them U4 XUTS-2205-0429, U5 W25Q16BVSSIG

Commit message: Add files via upload
Parts:
- added C21, C22: 22uF, Capacitor_SMD:C_0805_2012Metric, symbol Device:C
Connections:
- net GND: now also C21.2, C22.2
- net VBUS: now also C21.1, C22.1
