File: VL716.kicad_sch (KiCad schematic)
At the start: 28 parts, among them U1 VL716-Q4, Y1 25Mhz Crystal

Commit message: Add files via upload
Parts:
- removed C23, C24: 100nF, Capacitor_SMD:C_0402_1005Metric, symbol Device:C_Small
- added C29, C30: 100nF, Capacitor_SMD:C_0402_1005Metric, symbol Device:C_Small
Connections:
- net SARXVDD12 is gone; now on net +1V2: U1.5 (SARXVDD12)
- net SATXVDD12 is gone; now on net +1V2: U1.8 (SATXVDD12)
- net USB3RXVDD12 is gone; now on net +1V2: C26.2, U1.24 (U3RXVDD12)
- net USB3TXVDD12 is gone; now on net +1V2: C25.2, U1.19 (U3TXVDD12)
- net GND: now also C29.2, C30.2
- net +1V2: now reaches C11.1, C16.1, L1.1, U1.39 (DCVCC12)
- net +1V2: now also C17.1, C5.2, U1.14 (OSCVDD12), U1.30 (VDD12I), C29.1, C30.1
Other:
- moved on the sheet: C1, C10, C11, C16, C17, C18, C19, C2, C20, C25, C26, C3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
